File: mirte-pioneer/mirte_combination.kicad_pcb (KiCad board)
At the start: 2 copper layers, 55.6 x 81.9 mm, 49 parts, among them J1 Servo3, J10 IR1, J11 Conn_01x13_Female, J12 IR Object Detector 1, J14 IR2, J17 MC1, J18 MC2, J19 Servo1, J2 Conn_01x20_Female, J20 SRF1, J21 ENC2, J23 MC1-A, J24 MC1-B, J25 SRF2, J26 ENC1, J27 Servo2, J28 I2C2, J3 Servo4, J30 I2C1, J33 line out left, J34 Power in, J35 Power out, J37 on/off, J4 Conn_01x20_Female, J5 Conn_01x06_Pin, J7 Keypad, J8 Conn_01x06_Female, J9 IR Object Detector 2, Q1 DMG2305UX, Q2 DMN2050L, SW1 on/off, U1 CH340C, U2 CH340E

Commit message: test usb c pioneer pcb
Parts:
- removed J34: Power in, lcsc:MICRO-USB-SMD_U254-051T-4BH83-S1S
- added R1: 10k, Resistor_SMD:R_1206_3216Metric, F.Cu at (117.1, 59.3)
- added R12: 10k, Resistor_SMD:R_1206_3216Metric, F.Cu at (119.8, 62.2)
- added USB1: TYPE-C 16PIN 2MD(073), lcsc:USB-C-SMD_TYPE-C-6PIN-2MD-073, F.Cu at (118.8, 53.1)
Routing:
- net GND: track 42.1 -> 54.0 mm
- net Net-(USB1-CC1): track 0.00 -> 7.40 mm, vias 0 -> 2
- net Net-(USB1-CC2): track 0.00 -> 4.89 mm, vias 0 -> 2
- net 5V: track 336.6 -> 339.7 mm
- net D_GND: track 69.2 -> 71.2 mm, vias 13 -> 15
- added copper zone on F.Cu, net GND
