File: mirte-master/mirte-master.kicad_pcb (KiCad board)
At the start: 4 copper layers, 90.1 x 80.1 mm, 38 parts, among them J10 IMU MPU-9250, J11 Conn_01x03_Pin, J12 Conn_01x03_Pin, J13 sc, J14 sc, J16 sc, J17 sc, J18 sc, J19 sc, J20 sc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

Commit message: start update no modules
Parts:
- removed C4: 100nF, Capacitor_SMD:C_0805_2012Metric
- removed J10: IMU MPU-9250, Library:MPU9250
- removed J11: Conn_01x03_Pin, Connector_JST:JST_XH_B3B-XH-A_1x03_P2.50mm_Vertical
- removed J20, J21, J22: sc, easyeda:CONN-TH_XY126V-5.0-2P
- removed J7: INA226, Connector_JST:JST_XH_B4B-XH-A_1x04_P2.50mm_Vertical
- removed R1: 680, Resistor_SMD:R_0805_2012Metric
- added U1: PCA9685PW, Package_SO:TSSOP-28_4.4x9.7mm_P0.65mm, F.Cu at (69.3, 97.7)
- added U2: DRV8251DDAR, easyeda:SO-8_L4.9-W3.9-P1.27-LS6.0-BL-EP, F.Cu at (60.1, 117.7)
- added U3: DRV8251DDAR, easyeda:SO-8_L4.9-W3.9-P1.27-LS6.0-BL-EP, F.Cu at (66.6, 117.7)
- added U4: DRV8251DDAR, easyeda:SO-8_L4.9-W3.9-P1.27-LS6.0-BL-EP, F.Cu at (73.2, 117.7)
- added U5: DRV8251DDAR, easyeda:SO-8_L4.9-W3.9-P1.27-LS6.0-BL-EP, F.Cu at (79.7, 117.7)
- J8: value oled_conn -> IMU MPU-9250; footprint Connector_JST:JST_XH_B4B-XH-A_1x04_P2.50mm_Vertical -> Library:MPU9250
- J9: value pca9685 -> oled_conn; footprint Connector_PinHeader_2.54mm:PinHeader_1x06_P2.54mm_Vertical -> Connector_JST:JST_XH_B4B-XH-A_1x04_P2.50mm_Vertical
- moved J8 89.5 mm to (48.1, 84.6), turned to 0 degrees
- moved J9 64.1 mm to (68.4, 85.7), turned to 0 degrees
Connections:
- net /RX renamed /TX
- J8 pad 1: -BATT -> +5V
- J8 pad 2: +5V -> -BATT
- J9 pad 2: -BATT -> +5V
