File: mirte-master/pca9685.kicad_sch (KiCad schematic)
At the start: 1 part, among them J10 pca9685

Commit message: start update no modules
Parts:
- added U1: PCA9685PW, Package_SO:TSSOP-28_4.4x9.7mm_P0.65mm, symbol Driver_LED:PCA9685PW
- added U2, U3, U4, U5: DRV8251DDAR, easyeda:SO-8_L4.9-W3.9-P1.27-LS6.0-BL-EP, symbol easyeda:DRV8251DDAR
- J10: now left out of the parts list
Connections:
- net +5V: now also U1.28 (VDD)
- net GND: now also U1.14 (VSS), U1.23 (~{OE})
- net pca.SCL: now also U1.26 (SCL)
- net pca.SDA: now also U1.27 (SDA)
