File: mirte-master-power-input/diode.kicad_sch (KiCad schematic)
At the start: 6 parts, among them Q1 DMMT5401, Q2 SiA483DJ

Commit message: Power input: fix layout & fix diode setup
Parts:
- removed D1: LED, LED_SMD:LED_0805_2012Metric, symbol Device:LED
- removed R1: 10k, Resistor_SMD:R_0805_2012Metric, symbol Device:R
Connections:
- net MOS_Sig: now reaches Q1.4 (C2), Q2.3 (G), R3.1
